Commit message: fix laser tf

File: urdf/omni_base.xacro (robot description, xacro)
@@ -19,5 +19,5 @@
 	<xacro:omni_base_sim/>
 	<!-- Laser  -->
-	<xacro:include filename="$(find gazebo_plugins)/test/multi_robot_scenario/xacro/laser/hokuyo.xacro"/>
-	<xacro:laser name="base_laser" parent="base_link" xyz="0.16 0 0.2" rpy="0 0 0" meshes="package://gazebo_plugins/test/multi_robot_scenario/meshes/laser"/>
+	<xacro:include filename="$(find omni_base)/urdf/omni_laser.xacro"/>
+	<xacro:omni_laser name="base_laser" parent="base_link" xyz="0.16 0 0.2" rpy="0 0 0" meshes="package://gazebo_plugins/test/multi_robot_scenario/meshes/laser"/>
 </robot>

File: urdf/omni_laser.xacro (robot description, xacro)
@@ -1,6 +1,5 @@
 <?xml version="1.0"?>
-<!--hokuyo-->
 <robot xmlns:xacro="http://www.ros.org/wiki/xacro">
-<xacro:macro name="laser" params="name parent xyz rpy meshes">
+<xacro:macro name="omni_laser" params="name parent xyz rpy meshes">
 	<link name="${name}">
 		<visual>
@@ -48,7 +47,6 @@
 		</ray>
 		<plugin name="laser" filename="libgazebo_ros_laser.so" >
-			<robotNamespace></robotNamespace>
-			<topicName>${name}/scan</topicName>
-			<frameName>${name}</frameName>
+			<topicName>/scan</topicName>
+			<frameName>base_laser</frameName>
 		</plugin>
 		<!--
@@ -61,2 +59,3 @@
 	</gazebo>
 </xacro:macro>
+</robot>
