Commit message: add base_control_node

File: urdf/omni_body.xacro (robot description, xacro)
@@ -111,4 +111,6 @@
 			<child link="front_wheel"/>
 			<origin rpy="0 0 0" xyz="0.2 0 -0.08"/>
+    			<limit effort="100" velocity="100"/>
+    			<joint_properties damping="0.0" friction="0.0"/>
 		</joint>
 		<joint name="base_to_left_wheel" type="fixed">
@@ -116,4 +118,6 @@
 			<child link="left_wheel"/>
 			<origin rpy="0 0 0" xyz="-0.1 0.1732 -0.08"/>
+	    		<limit effort="100" velocity="100"/>
+    			<joint_properties damping="0.0" friction="0.0"/>
 		</joint>
 		<joint name="base_to_right_wheel" type="fixed">
@@ -121,4 +125,6 @@
 			<child link="right_wheel"/>
 			<origin rpy="0 0 0" xyz="-0.1 -0.1732 -0.08"/>
+		    	<limit effort="100" velocity="100"/>
+    			<joint_properties damping="0.0" friction="0.0"/>
 		</joint>
 	</xacro:macro>
